File: Voltage_Indicator/RM28_Voltage_Indicator_V1.0.kicad_pcb (KiCad board)
At the start: 2 copper layers, 44 x 16.5 mm, 21 parts, among them IC1 NCP785AH120T1G, J1 Molex_Micro-Fit_3.0_43650-020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, J2 Molex_Micro-Fit_3.0_43650-020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, Q1 SBCP56-16T1G, U1 1SMB5927BT3G

Commit message: Final layout changes
Parts:
- removed the REF** at (126.3, 59.1)
- added G***: LOGO, RM:RM_logo_medium, F.Cu at (128.6, 57.0)
- added G***: LOGO, RM:HV_Triangle, F.Cu at (104.2, 58.0)
- R8: value 500Ω -> 1kΩ
Routing:
- net (no net): track 2.20 -> 0.00 mm
Other:
- outline, holes or cut-outs redrawn
